File: GSR/GSRv2.1.sch (EAGLE design)
At the start: 38 parts, among them U1 ARDUINO_MINI

Commit message: fixed errors and aligned board
Connections:
- removed net N$7: POWER.2
- net GND: now also POWER.2
Changed lines of the file:
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@@
 <pinref part="GND1" gate="1" pin="GND"/>
 <wire x1="-0.254" y1="142.24" x2="3.556" y2="142.24" width="0.1524" layer="91"/>
-<pinref part="C3" gate="G$1" pin="-"/>
 <wire x1="3.556" y1="142.24" x2="9.652" y2="142.24" width="0.1524" layer="91"/>
-<wire x1="9.652" y1="144.78" x2="9.652" y2="142.24" width="0.1524" layer="91"/>
 <pinref part="C1" gate="G$1" pin="-"/>
 <wire x1="3.556" y1="144.78" x2="3.556" y2="142.24" width="0.1524" layer="91"/>
 <junction x="3.556" y="142.24"/>
+<pinref part="C3" gate="G$1" pin="-"/>
+<wire x1="9.652" y1="142.24" x2="9.652" y2="144.78" width="0.1524" layer="91"/>
+<pinref part="POWER" gate="G$1" pin="2"/>
+<wire x1="9.652" y1="142.24" x2="25.146" y2="142.24" width="0.1524" layer="91"/>
+<junction x="9.652" y="142.24"/>
 </segment>
 <segment>
@@
 </segment>
 </net>
-<net name="N$7" class="0">
-<segment>
-<pinref part="POWER" gate="G$1" pin="2"/>
-<wire x1="9.652" y1="142.24" x2="25.146" y2="142.24" width="0.1524" layer="91"/>
-</segment>
-</net>
